Commit message: Add chessboard model and white color extractiongit status!

File: mybot_description/urdf/mybot.xacro (robot description, xacro)
@@ -160,5 +160,5 @@
   <joint name="camera_joint" type="fixed">
     <axis xyz="0 1 0" />
-    <origin xyz=".2 0 0" rpy="0 0 0"/>
+    <origin xyz=".2 0 0.3" rpy="0 0 0"/>
     <parent link="chassis"/>
     <child link="camera"/>

Commit message: Add perspective and log polar transforms

File: mybot_description/urdf/mybot.xacro (robot description, xacro)
@@ -160,5 +160,5 @@
   <joint name="camera_joint" type="fixed">
     <axis xyz="0 1 0" />
-    <origin xyz=".2 0 0.3" rpy="0 0 0"/>
+    <origin xyz=".2 0 2" rpy="0 0.5 0"/>
     <parent link="chassis"/>
     <child link="camera"/>

Commit message: Testing lower camera position

File: mybot_description/urdf/mybot.xacro (robot description, xacro)
@@ -160,5 +160,5 @@
   <joint name="camera_joint" type="fixed">
     <axis xyz="0 1 0" />
-    <origin xyz=".2 0 2" rpy="0 0.5 0"/>
+    <origin xyz=".2 0 0.5" rpy="0 0.5 0"/>
     <parent link="chassis"/>
     <child link="camera"/>
